File: Mau Keys.kicad_pcb (KiCad board)
At the start: 2 copper layers, 257 x 220.2 mm, 68 parts

Commit message: detallitos
Parts:
- removed the NNV2 at (153.4, 157.4)
- removed NNV2_R1: ~, Microcontroller:nice_nano
- removed the RSW1 at (159.0, 192.0)
- removed the SW_POWER1 at (153.4, 157.4)
- NNV2: moved to F.Cu
- moved Switch13 171.7 mm to (219.0, 67.0)
- moved Switch3 171.7 mm to (219.0, 27.0)
- moved Switch8 171.7 mm to (219.0, 47.0)
- moved Switch10 17.0 mm to (179.0, 60.0)
- moved Switch14 17.0 mm to (199.0, 77.0)
- moved Switch15 17.0 mm to (179.0, 80.0)
- moved Switch4 17.0 mm to (199.0, 37.0)
- moved Switch5 17.0 mm to (179.0, 40.0)
- moved Switch9 17.0 mm to (199.0, 57.0)
- moved SW_POWER2 11.7 mm to (159.4, 40.0)
- moved NNV2 0.86 mm to (159.4, 40.0), turned to 0 degrees
Routing:
- net S11: track 305.3 -> 152.6 mm
- net S1: track 289.4 -> 144.7 mm
- net S6: track 274.3 -> 137.1 mm
- net S12: track 240.2 -> 120.1 mm
- net S2: track 226.5 -> 113.2 mm
- net S7: track 212.4 -> 106.2 mm
- net S13: track 178.9 -> 89.4 mm
- net S3: track 175.5 -> 87.7 mm
- net S8: track 160.6 -> 80.3 mm
- net S14: track 133.0 -> 66.5 mm
- net S4: track 126.2 -> 63.1 mm
- net S16: track 116.3 -> 58.2 mm
- net S9: track 114.3 -> 57.2 mm
- net S17: track 95.1 -> 47.6 mm
- net S5: track 87.3 -> 43.7 mm
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Other:
- board size 257 x 220.2 mm -> 256.2 x 102.8 mm

Commit message: fix switch fp
Parts:
- removed the Switch1 at (47.5, 174.3)
- removed the Switch11 at (55.8, 213.4)
- removed the Switch12 at (73.8, 196.4)
- removed the Switch14 at (113.8, 194.4)
- removed the Switch16 at (122.6, 217.5)
- removed the Switch17 at (143.5, 223.1)
- removed the Switch17 at (230.0, 109.8)
- removed the Switch2 at (70.3, 156.6)
- removed the Switch4 at (113.8, 154.4)
- removed the Switch6 at (51.6, 193.9)
- removed the Switch7 at (72.0, 176.5)
- removed the Switch9 at (113.8, 174.4)
- removed the SwitchR_1 at (230.0, 119.3)
- removed the SwitchR_11 at (242.6, 147.9)
- removed the SwitchR_12 at (242.6, 157.5)
- removed the SwitchR_13 at (256.0, 75.0)
- removed the SwitchR_14 at (255.2, 109.8)
- removed the SwitchR_16 at (255.2, 128.8)
- removed the SwitchR_2 at (230.0, 128.8)
- removed the SwitchR_3 at (230.0, 138.4)
- removed the SwitchR_4 at (230.0, 147.9)
- removed the SwitchR_6 at (237.0, 72.0)
- removed the SwitchR_7 at (242.6, 109.8)
- removed the SwitchR_8 at (242.6, 119.3)
- removed the SwitchR_9 at (242.6, 128.8)
- added G***: LOGO, graphics:logoprojectmauskeys, F.Cu at (79.8, 90.6)
- added G***: LOGO, graphics:logoprojectmauskeys, F.Cu at (218.0, 90.0)
- added SwitchR_17: ~, Switches:keyswitch_cherrymx_alps_choc12_slots_1u, F.Cu at (190.1, 100.1)
- SW_POWER1: moved to F.Cu
- moved SwitchR_4 160.6 mm to (242.5, 39.2), turned to -5 degrees
- moved SwitchR_9 159.5 mm to (240.7, 59.2), turned to -5 degrees
- moved SwitchR_14 158.4 mm to (239.0, 79.1), turned to -5 degrees
- moved SwitchR_5 106.6 mm to (265.3, 57.0), turned to -12 degrees
- moved SwitchR_10 64.6 mm to (261.2, 76.5), turned to -12 degrees
- moved RSW2 52.2 mm to (154.0, 75.0), turned to 90 degrees
- moved SwitchR_16 32.7 mm to (169.2, 105.7), turned to 19.35 degrees
- moved SwitchR_15 23.3 mm to (257.0, 96.1), turned to -12 degrees
- moved RSW1 0.56 mm to (145.0, 75.0)
- turned SW_POWER1 to 0 degrees
- turned Switch17 to -19.35 degrees
- renumbered NNV2 to NNV2_R1, Switch5 to SwitchR_1, Switch15 to SwitchR_11, Switch14 to SwitchR_12, Switch13 to SwitchR_13, Switch15 to SwitchR_14, SwitchR_17 to SwitchR_16, Switch4 to SwitchR_2, Switch3 to SwitchR_3, Switch5 to SwitchR_4, Switch10 to SwitchR_6, Switch9 to SwitchR_7, Switch8 to SwitchR_8, Switch10 to SwitchR_9
Connections:
- NNV2 pad 14: VBAT -> BAT+
- NNV2_R1 pad 10: S7 -> S11_R
- NNV2_R1 pad 11: S8 -> S17_R
- NNV2_R1 pad 12: S9 -> S16_R
- NNV2_R1 pad 13: S10 -> unconnected-(NNV2_R1-Pad13)
- NNV2_R1 pad 14: VBAT -> BAT+
- NNV2_R1 pad 19: S11 -> S5_R
- NNV2_R1 pad 2: S1 -> S9_R
- NNV2_R1 pad 20: S12 -> S4_R
- NNV2_R1 pad 21: S13 -> S3_R
- NNV2_R1 pad 22: S14 -> S2_R
- NNV2_R1 pad 23: S15 -> S1_R
- NNV2_R1 pad 24: S16 -> S10_R
- NNV2_R1 pad 25: S17 -> S8_R
- NNV2_R1 pad 26: unconnected-(NNV2-Pad26) -> S6_R
- NNV2_R1 pad 27: unconnected-(NNV2-Pad27) -> unconnected-(NNV2_R1-Pad27)
- NNV2_R1 pad 28: unconnected-(NNV2-Pad28) -> unconnected-(NNV2_R1-Pad28)
- NNV2_R1 pad 29: unconnected-(NNV2-Pad29) -> unconnected-(NNV2_R1-Pad29)
- NNV2_R1 pad 3: S2 -> S7_R
- NNV2_R1 pad 6: S3 -> S15_R
- NNV2_R1 pad 7: S4 -> S14_R
- NNV2_R1 pad 8: S5 -> S13_R
- NNV2_R1 pad 9: S6 -> S12_R
- SwitchR_1 pad 1: S5 -> S1_R
- SwitchR_11 pad 1: S15 -> S11_R
- SwitchR_12 pad 1: S14 -> S12_R
- SwitchR_13 pad 1: S13 -> S13_R
- SwitchR_14 pad 1: S15 -> S14_R
- SwitchR_16 pad 1: S17_R -> S16_R
- SwitchR_2 pad 1: S4 -> S2_R
- SwitchR_3 pad 1: S3 -> S3_R
- SwitchR_4 pad 1: S5 -> S4_R
- SwitchR_6 pad 1: S10 -> S6_R
- SwitchR_7 pad 1: S9 -> S7_R
- SwitchR_8 pad 1: S8 -> S8_R
- SwitchR_9 pad 1: S10 -> S9_R
Routing:
- net S15_R: track 0.00 -> 150.8 mm
- net S5_R: track 0.00 -> 147.1 mm
- net S9_R: track 0.00 -> 137.2 mm
- net S10_R: track 0.00 -> 129.6 mm
- net S14_R: track 0.00 -> 117.2 mm
- net S4_R: track 0.00 -> 113.8 mm
- net S7_R: track 0.00 -> 76.1 mm
- net S13_R: track 0.00 -> 72.4 mm
- net S3_R: track 0.00 -> 71.4 mm
- net S8_R: track 0.00 -> 61.1 mm
- net S2_R: track 0.00 -> 53.9 mm
- net S12_R: track 0.00 -> 52.5 mm
- net S17_R: track 0.00 -> 50.3 mm
- net S16_R: track 0.00 -> 46.8 mm
- net RESET: track 30.0 -> 61.4 mm, vias 2 -> 4
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- added copper zone on B.Cu, net GND
- added copper zone on F.Cu, net GND
