File: Mau Keys.kicad_pcb (KiCad board)
At the start: 2 copper layers, 256.2 x 102.8 mm, 42 parts

Commit message: fix switch traces
Parts:
- added REF**: MountingHole_3.2mm_M3_DIN965_Pad, reset:MountingHole_3.2mm_M3_DIN965_Pad, F.Cu at (25.5, 51.9)
- added REF**: MountingHole_3.2mm_M3_DIN965_Pad, reset:MountingHole_3.2mm_M3_DIN965_Pad, F.Cu at (81.0, 35.5)
- added REF**: MountingHole_3.2mm_M3_DIN965_Pad, reset:MountingHole_3.2mm_M3_DIN965_Pad, F.Cu at (140.5, 47.5)
- added REF**: MountingHole_3.2mm_M3_DIN965_Pad, reset:MountingHole_3.2mm_M3_DIN965_Pad, F.Cu at (133.1, 114.3)
- added REF**: MountingHole_3.2mm_M3_DIN965_Pad, reset:MountingHole_3.2mm_M3_DIN965_Pad, F.Cu at (80.0, 78.5)
- added REF**: MountingHole_3.2mm_M3_DIN965_Pad, reset:MountingHole_3.2mm_M3_DIN965_Pad, F.Cu at (143.3, 83.0)
- added REF**: MountingHole_3.2mm_M3_DIN965_Pad, reset:MountingHole_3.2mm_M3_DIN965_Pad, F.Cu at (37.0, 104.5)
Routing:
- net S1_R: track 25.4 -> 37.8 mm
- net S6_R: track 13.0 -> 24.3 mm
- net S3_R: track 71.4 -> 79.7 mm
- net S13_R: track 72.4 -> 80.6 mm
- net S8_R: track 61.1 -> 69.4 mm
- net S2_R: track 53.9 -> 57.7 mm
- net S11_R: track 28.4 -> 31.9 mm
- net S7_R: track 76.1 -> 79.6 mm
- net S12_R: track 52.5 -> 56.0 mm
- net S15_R: track 150.8 -> 148.0 mm
- net S9_R: track 137.2 -> 134.4 mm
- net S4_R: track 113.8 -> 115.4 mm
- net S5_R: track 147.1 -> 148.6 mm
- net S10_R: track 129.6 -> 128.3 mm
- net S16_R: track 46.8 -> 45.7 mm
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