File: Mau Keys.kicad_pcb (KiCad board)
At the start: 2 copper layers, 256.2 x 181.3 mm, 47 parts

Commit message: new arrangement
Parts:
- removed G*** (x2): LOGO, graphics:logoprojectmauskeys
- removed REF** (x5): MountingHole_3.2mm_M3_DIN965_Pad, reset:MountingHole_3.2mm_M3_DIN965_Pad
- added SwitchR_1: ~, Switches:keyswitch_cherrymx_alps_choc12_slots_1u, F.Cu at (185.7, -49.9)
- added SwitchR_10: ~, Switches:keyswitch_cherrymx_alps_choc12_slots_1u, F.Cu at (261.6, -12.7)
- added SwitchR_11: ~, Switches:keyswitch_cherrymx_alps_choc12_slots_1u, F.Cu at (185.7, -11.9)
- added SwitchR_12: ~, Switches:keyswitch_cherrymx_alps_choc12_slots_1u, F.Cu at (204.7, -14.9)
- added SwitchR_13: ~, Switches:keyswitch_cherrymx_alps_choc12_slots_1u, F.Cu at (223.7, -24.9)
- added SwitchR_14: ~, Switches:keyswitch_cherrymx_alps_choc12_slots_1u, F.Cu at (242.2, -10.9)
- added SwitchR_15: ~, Switches:keyswitch_cherrymx_alps_choc12_slots_1u, F.Cu at (258.7, 6.10)
- added SwitchR_16: ~, Switches:keyswitch_cherrymx_alps_choc12_slots_1u, F.Cu at (179.0, 11.1)
- added SwitchR_17: ~, Switches:keyswitch_cherrymx_alps_choc12_slots_1u, F.Cu at (197.7, 8.11)
- added SwitchR_2: ~, Switches:keyswitch_cherrymx_alps_choc12_slots_1u, F.Cu at (204.7, -52.9)
- added SwitchR_3: ~, Switches:keyswitch_cherrymx_alps_choc12_slots_1u, F.Cu at (223.7, -62.9)
- added SwitchR_4: ~, Switches:keyswitch_cherrymx_alps_choc12_slots_1u, F.Cu at (245.5, -48.7)
- added SwitchR_5: ~, Switches:keyswitch_cherrymx_alps_choc12_slots_1u, F.Cu at (264.4, -31.5)
- added SwitchR_6: ~, Switches:keyswitch_cherrymx_alps_choc12_slots_1u, F.Cu at (185.7, -30.9)
- added SwitchR_7: ~, Switches:keyswitch_cherrymx_alps_choc12_slots_1u, F.Cu at (204.7, -33.9)
- added SwitchR_8: ~, Switches:keyswitch_cherrymx_alps_choc12_slots_1u, F.Cu at (223.7, -43.9)
- added SwitchR_9: ~, Switches:keyswitch_cherrymx_alps_choc12_slots_1u, F.Cu at (243.9, -29.8)
- moved Switch17 94.8 mm to (124.8, 11.0), turned to -9 degrees
- moved Switch16 92.1 mm to (106.0, 8.00), turned to -9 degrees
- moved Switch15 92.0 mm to (118.0, -12.0)
- moved Switch14 92.0 mm to (99.0, -15.0)
- moved Switch13 92.0 mm to (80.0, -25.0)
- moved Switch10 91.0 mm to (118.0, -31.0)
- moved Switch9 91.0 mm to (99.0, -34.0)
- moved Switch8 91.0 mm to (80.0, -44.0)
- moved RSW2 90.6 mm to (161.5, -15.2)
- moved RSW1 90.3 mm to (142.2, -15.2)
- moved NNV2_R1 90.1 mm to (166.1, -49.9)
- moved SW_POWER2 90.1 mm to (166.1, -49.9)
- moved Switch11 90.0 mm to (45.0, 6.00), turned to 8.6 degrees
- moved NNV2 90.0 mm to (137.6, -50.0)
- moved SW_POWER1 90.0 mm to (137.6, -50.0)
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Routing:
- net S5_R: track 148.6 -> 289.3 mm
- net S6: track 128.3 -> 116.7 mm
- net S8: track 72.0 -> 63.8 mm
- net S3: track 79.4 -> 71.9 mm
- net S11: track 143.8 -> 136.7 mm
- net S10: track 31.7 -> 24.7 mm
- net S1: track 136.8 -> 132.0 mm
- net S4: track 54.8 -> 50.2 mm
- net S7: track 97.6 -> 93.1 mm
- net S9: track 48.8 -> 44.4 mm
- net S2: track 105.1 -> 101.4 mm
- net S5: track 35.3 -> 32.1 mm
- net S13: track 81.1 -> 78.3 mm
- net S14: track 58.1 -> 55.4 mm
- net S12: track 111.7 -> 110.1 mm
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- removed copper zone on B.Cu, net GND
- removed copper zone on F.Cu, net GND
Other:
- board size 256.2 x 181.3 mm -> 246.4 x 94.3 mm

Commit message: pcb casi terminado
Parts:
- removed the SwitchR_1 at (179.0, 40.0)
- removed the SwitchR_10 at (261.2, 76.5)
- removed the SwitchR_11 at (179.0, 80.0)
- removed the SwitchR_12 at (199.0, 77.0)
- removed the SwitchR_13 at (219.0, 67.0)
- removed the SwitchR_14 at (239.0, 79.1)
- removed the SwitchR_15 at (257.0, 96.1)
- removed the SwitchR_16 at (169.2, 105.7)
- removed the SwitchR_17 at (190.1, 100.1)
- removed the SwitchR_2 at (199.0, 37.0)
- removed the SwitchR_3 at (219.0, 27.0)
- removed the SwitchR_4 at (242.5, 39.2)
- removed the SwitchR_5 at (265.3, 57.0)
- removed the SwitchR_6 at (179.0, 60.0)
- removed the SwitchR_7 at (199.0, 57.0)
- removed the SwitchR_8 at (219.0, 47.0)
- removed the SwitchR_9 at (240.7, 59.2)
- added G***: LOGO, graphics:logo_pcb_hands, F.Cu at (80.0, 113.8)
- added G***: LOGO, graphics:logo_pcb_hands, F.Cu at (222.2, 114.3)
- moved RSW1 116.9 mm to (139.7, 101.6)
- moved RSW2 116.8 mm to (162.6, 101.6)
- moved NNV2 116.0 mm to (137.2, 66.0)
- moved SW_POWER1 116.0 mm to (137.2, 66.0)
- moved Switch10 116.0 mm to (117.5, 85.0)
- moved Switch11 116.0 mm to (44.6, 122.0)
- moved Switch13 116.0 mm to (79.5, 91.0)
- moved Switch14 116.0 mm to (98.5, 101.0)
- moved Switch15 116.0 mm to (117.5, 104.0)
- moved Switch16 116.0 mm to (105.5, 124.0)
- moved Switch5 116.0 mm to (117.5, 66.0)
- moved Switch6 116.0 mm to (41.7, 103.3)
- moved Switch7 116.0 mm to (59.4, 86.1)
- moved Switch8 116.0 mm to (79.5, 72.0)
- moved Switch9 116.0 mm to (98.5, 82.0)
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Routing:
- net S5_R: track 289.3 -> 140.7 mm
- net S11_R: track 31.9 -> 46.6 mm
- net S16_R: track 45.7 -> 35.4 mm
- net S12_R: track 56.0 -> 65.5 mm
- net S15_R: track 148.0 -> 140.1 mm
- net S9_R: track 134.4 -> 127.2 mm
- net S13_R: track 80.6 -> 87.4 mm
- net S10_R: track 128.3 -> 122.5 mm
- net S17_R: track 49.3 -> 55.0 mm
- net S4_R: track 115.4 -> 111.3 mm
- net S7_R: track 79.6 -> 77.8 mm
- net S6_R: track 24.3 -> 26.1 mm
- net S8_R: track 69.4 -> 67.7 mm
- net S2_R: track 57.7 -> 56.6 mm
- net RESET: track 60.4 -> 59.2 mm
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- added copper zone on B.Cu, net GND
- added copper zone on F.Cu, net GND
Other:
- board size 246.4 x 94.3 mm -> 245.8 x 94.2 mm

Commit message: pcb final
Parts:
- added G***: LOGO, LOGO, F.Cu at (222.2, 114.3)
- added G***: LOGO, LOGO, F.Cu at (82.5, 113.8)
- added REF**: MountingHole_2.2mm_M2_DIN965_Pad, MountingHole:MountingHole_2.2mm_M2_DIN965_Pad, F.Cu at (52.1, 78.5)
- added REF**: MountingHole_2.2mm_M2_DIN965_Pad, MountingHole:MountingHole_2.2mm_M2_DIN965_Pad, F.Cu at (39.4, 94.0)
- added REF**: MountingHole_2.2mm_M2_DIN965_Pad, MountingHole:MountingHole_2.2mm_M2_DIN965_Pad, F.Cu at (108.7, 109.7)
- added REF**: MountingHole_2.2mm_M2_DIN965_Pad, MountingHole:MountingHole_2.2mm_M2_DIN965_Pad, F.Cu at (131.8, 133.3)
- added REF**: MountingHole_2.2mm_M2_DIN965_Pad, MountingHole:MountingHole_2.2mm_M2_DIN965_Pad, F.Cu at (66.0, 123.2)
- added REF**: MountingHole_2.2mm_M2_DIN965_Pad, MountingHole:MountingHole_2.2mm_M2_DIN965_Pad, F.Cu at (135.9, 110.5)
- added REF**: MountingHole_2.2mm_M2_DIN965_Pad, MountingHole:MountingHole_2.2mm_M2_DIN965_Pad, F.Cu at (139.7, 73.7)
- added REF**: MountingHole_2.2mm_M2_DIN965_Pad, MountingHole:MountingHole_2.2mm_M2_DIN965_Pad, B.Cu at (266.7, 93.5)
- added REF**: MountingHole_2.2mm_M2_DIN965_Pad, MountingHole:MountingHole_2.2mm_M2_DIN965_Pad, B.Cu at (262.9, 111.5)
- added REF**: MountingHole_2.2mm_M2_DIN965_Pad, MountingHole:MountingHole_2.2mm_M2_DIN965_Pad, B.Cu at (252.7, 78.5)
- added REF**: MountingHole_2.2mm_M2_DIN965_Pad, MountingHole:MountingHole_2.2mm_M2_DIN965_Pad, B.Cu at (194.3, 108.7)
- added REF**: OSHW-Symbol_6.7x6mm_Copper, Symbol:OSHW-Symbol_6.7x6mm_Copper, F.Cu at (57.4, 125.0)
- added REF**: MountingHole_2.2mm_M2_DIN965_Pad, MountingHole:MountingHole_2.2mm_M2_DIN965_Pad, B.Cu at (194.3, 69.3)
- added REF**: MountingHole_2.2mm_M2_DIN965_Pad, MountingHole:MountingHole_2.2mm_M2_DIN965_Pad, B.Cu at (238.8, 123.2)
- added REF**: MountingHole_2.2mm_M2_DIN965_Pad, MountingHole:MountingHole_2.2mm_M2_DIN965_Pad, B.Cu at (178.6, 132.8)
- added REF**: MountingHole_2.2mm_M2_DIN965_Pad, MountingHole:MountingHole_2.2mm_M2_DIN965_Pad, B.Cu at (208.3, 125.7)
- added REF**: MountingHole_2.2mm_M2_DIN965_Pad, MountingHole:MountingHole_2.2mm_M2_DIN965_Pad, B.Cu at (212.6, 93.7)
- added REF**: MountingHole_2.2mm_M2_DIN965_Pad, MountingHole:MountingHole_2.2mm_M2_DIN965_Pad, B.Cu at (168.9, 110.5)
- added REF**: MountingHole_2.2mm_M2_DIN965_Pad, MountingHole:MountingHole_2.2mm_M2_DIN965_Pad, B.Cu at (234.2, 95.8)
- added REF**: MountingHole_2.2mm_M2_DIN965_Pad, MountingHole:MountingHole_2.2mm_M2_DIN965_Pad, B.Cu at (222.8, 60.7)
- added REF**: MountingHole_2.2mm_M2_DIN965_Pad, MountingHole:MountingHole_2.2mm_M2_DIN965_Pad, B.Cu at (165.1, 73.7)
- added REF**: MountingHole_2.2mm_M2_DIN965_Pad, MountingHole:MountingHole_2.2mm_M2_DIN965_Pad, F.Cu at (107.4, 70.6)
- added REF**: MountingHole_2.2mm_M2_DIN965_Pad, MountingHole:MountingHole_2.2mm_M2_DIN965_Pad, F.Cu at (92.2, 93.7)
- added REF**: MountingHole_2.2mm_M2_DIN965_Pad, MountingHole:MountingHole_2.2mm_M2_DIN965_Pad, F.Cu at (70.6, 95.8)
- added REF**: MountingHole_2.2mm_M2_DIN965_Pad, MountingHole:MountingHole_2.2mm_M2_DIN965_Pad, F.Cu at (43.2, 113.0)
- added REF**: MountingHole_2.2mm_M2_DIN965_Pad, MountingHole:MountingHole_2.2mm_M2_DIN965_Pad, F.Cu at (96.5, 125.7)
- added REF**: MountingHole_2.2mm_M2_DIN965_Pad, MountingHole:MountingHole_2.2mm_M2_DIN965_Pad, F.Cu at (82.0, 60.7)
- added REF**: OSHW-Symbol_6.7x6mm_Copper, Symbol:OSHW-Symbol_6.7x6mm_Copper, F.Cu at (245.9, 124.5)
- moved RSW1 2.54 mm to (142.2, 101.6)
- moved Switch17 2.54 mm to (126.8, 127.0)
- moved Switch1 2.54 mm to (41.4, 84.5)
- moved Switch11 2.54 mm to (47.1, 122.0)
- moved Switch12 2.54 mm to (63.6, 105.0)
- moved Switch2 2.54 mm to (60.3, 67.2)
- moved Switch6 2.54 mm to (44.3, 103.3)
- moved Switch7 2.54 mm to (61.9, 86.1)
- moved G*** 2.54 mm to (82.5, 113.8)
- moved NNV2 2.54 mm to (139.7, 66.0)
- moved SW_POWER1 2.54 mm to (139.7, 66.0)
- moved Switch10 2.54 mm to (120.1, 85.0)
- moved Switch13 2.54 mm to (82.1, 91.0)
- moved Switch14 2.54 mm to (101.1, 101.0)
- moved Switch15 2.54 mm to (120.1, 104.0)
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Routing:
- net S16_R: track 35.4 -> 42.9 mm
- net S17: track 40.7 -> 37.7 mm
- net S9_R: track 127.2 -> 129.0 mm
- net S9: track 44.4 -> 42.8 mm
- net S6: track 116.7 -> 115.2 mm
- net S7_R: track 77.8 -> 79.3 mm
- net S7: track 93.1 -> 91.8 mm
- net S14: track 55.4 -> 56.5 mm
- net S16: track 50.5 -> 49.5 mm
- net S12: track 110.1 -> 111.1 mm
- net S11: track 136.7 -> 137.7 mm
- net S13: track 78.3 -> 79.3 mm
- net S10_R: track 122.5 -> 121.8 mm
Other:
- board size 245.8 x 94.2 mm -> 243.3 x 94.2 mm
